File: shield/PTL-ino-prog_avr_pic/_saved_PTL-ino-prog_avr_pic.sch (KiCad schematic (older format))
At the start: 30 parts, among them P1 CONN_8, P2 CONN_6, P3 CONN_10, P4 CONN_8, P5 CONN_3X2, P6 CONN_01X02, P7 CONN_6, Q1 BC548, U1 PIC16F1455, U2 ATmega328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

Commit message: added quartz
Parts:
- RST1, USR1, USR2: footprint Buttons_Switches_ThroughHole:SW_PUSH_SMALL -> PTL-ino:SW_PUSH_SMALL
Changed lines of the file:
@@
 F 0 "RST1" H 3750 5710 50  0000 C CNN
 F 1 "RST" H 3600 5520 50  0000 C CNN
-F 2 "Buttons_Switches_ThroughHole:SW_PUSH_SMALL" H 3600 5600 60  0001 C CNN
+F 2 "PTL-ino:SW_PUSH_SMALL" H 3600 5600 60  0001 C CNN
 F 3 "" H 3600 5600 60  0000 C CNN
 	1    3600 5600
@@
 F 0 "USR2" H 11050 3510 50  0000 C CNN
 F 1 "SW_PUSH" H 10900 3320 50  0000 C CNN
-F 2 "Buttons_Switches_ThroughHole:SW_PUSH_SMALL" H 10900 3400 60  0001 C CNN
+F 2 "PTL-ino:SW_PUSH_SMALL" H 10900 3400 60  0001 C CNN
 F 3 "" H 10900 3400 60  0000 C CNN
 	1    10900 3400
@@
 F 0 "USR1" H 10650 3510 50  0000 C CNN
 F 1 "SW_PUSH" H 10500 3320 50  0000 C CNN
-F 2 "Buttons_Switches_ThroughHole:SW_PUSH_SMALL" H 10500 3400 60  0001 C CNN
+F 2 "PTL-ino:SW_PUSH_SMALL" H 10500 3400 60  0001 C CNN
 F 3 "" H 10500 3400 60  0000 C CNN
 	1    10500 3400
